File: Hardware/F-91wa.sch (EAGLE design)
At the start: 14 parts

Commit message: This is for the third week
Parts:
- added U$1: LSM6DS3_CAST, LinnesLab-Sensors:LSM6DS3_CAST
- added U1: (no value), LinnesLab-Microcontrollers:ARTEMIS.CAST
Connections:
- new net SCLA: U$1.SCL
- new net SDA: U$1.SDA
- net 3.3V: now also U$1.VCC
- net GND: now also U$1.GND
Changed lines of the file:
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@@
 <part name="GND9" library="LinnesLab-Symbols" deviceset="GND" device=""/>
 <part name="SUPPLY4" library="LinnesLab-Symbols" deviceset="VLIPO" device=""/>
+<part name="U$1" library="LinnesLab-Sensors" deviceset="LSM6DS3_CAST" device=""/>
+<part name="U1" library="LinnesLab-Microcontrollers" deviceset="ARTEMIS.CAST" device=""/>
+<part name="SUPPLY6" library="LinnesLab-Symbols" deviceset="3.3V" device=""/>
+<part name="GND10" library="LinnesLab-Symbols" deviceset="GND" device=""/>
 </parts>
 <sheets>
@@
 </instance>
 <instance part="SUPPLY1" gate="G$1" x="149.86" y="53.34" smashed="yes">
-<attribute name="VALUE" x="149.86" y="56.134" size="1.778" layer="96" align="bottom-center"/>
+<attribute name="VALUE" x="149.86" y="55.88" size="1.778" layer="96" align="bottom-center"/>
 </instance>
 <instance part="SUPPLY2" gate="G$1" x="73.66" y="25.4" smashed="yes">
@@
 <instance part="SUPPLY4" gate="G$1" x="162.56" y="48.26" smashed="yes">
 <attribute name="VALUE" x="162.56" y="51.054" size="1.778" layer="96" align="bottom-center"/>
+</instance>
+<instance part="U$1" gate="G$1" x="195.58" y="50.8" smashed="yes">
+<attribute name="NAME" x="187.96" y="55.88" size="1.778" layer="95"/>
+<attribute name="VALUE" x="187.96" y="43.18" size="1.778" layer="96"/>
+</instance>
+<instance part="U1" gate="G$1" x="208.28" y="-5.08" smashed="yes">
+<attribute name="NAME" x="177.8" y="36.068" size="1.778" layer="95"/>
+<attribute name="VALUE" x="177.8" y="-53.34" size="1.778" layer="96"/>
+</instance>
+<instance part="SUPPLY6" gate="G$1" x="175.26" y="60.96" smashed="yes">
+<attribute name="VALUE" x="175.26" y="63.754" size="1.778" layer="96" align="bottom-center"/>
+</instance>
+<instance part="GND10" gate="G$1" x="177.8" y="43.18" smashed="yes">
+<attribute name="VALUE" x="177.8" y="42.926" size="1.778" layer="96" align="top-center"/>
 </instance>
 </instances>
@@
 <pinref part="GND9" gate="G$1" pin="GND"/>
 <wire x1="162.56" y1="20.32" x2="162.56" y2="17.78" width="0.1524" layer="91"/>
+</segment>
+<segment>
+<pinref part="U$1" gate="G$1" pin="GND"/>
+<wire x1="182.88" y1="53.34" x2="177.8" y2="53.34" width="0.1524" layer="91"/>
+<wire x1="177.8" y1="53.34" x2="177.8" y2="45.72" width="0.1524" layer="91"/>
+<pinref part="GND10" gate="G$1" pin="GND"/>
 </segment>
 </net>
@@
 <wire x1="149.86" y1="48.26" x2="149.86" y2="53.34" width="0.1524" layer="91"/>
 <junction x="149.86" y="48.26"/>
+</segment>
+<segment>
+<pinref part="U$1" gate="G$1" pin="VCC"/>
+<wire x1="182.88" y1="48.26" x2="175.26" y2="48.26" width="0.1524" layer="91"/>
+<wire x1="175.26" y1="48.26" x2="175.26" y2="60.96" width="0.1524" layer="91"/>
+<pinref part="SUPPLY6" gate="G$1" pin="3.3V"/>
 </segment>
 </net>
@@
 </segment>
 </net>
+<net name="SDA" class="0">
+<segment>
+<pinref part="U$1" gate="G$1" pin="SDA"/>
+<wire x1="208.28" y1="53.34" x2="215.9" y2="53.34" width="0.1524" layer="91"/>
+<label x="215.9" y="53.34" size="1.778" layer="95"/>
+</segment>
+</net>
+<net name="SCLA" class="0">
+<segment>
+<pinref part="U$1" gate="G$1" pin="SCL"/>
+<wire x1="208.28" y1="48.26" x2="215.9" y2="48.26" width="0.1524" layer="91"/>
+<label x="215.9" y="48.26" size="1.778" layer="95"/>
+</segment>
+</net>
